Commit message: Update ridgeback.urdf.xacro

File: ridgeback_description/urdf/ridgeback.urdf.xacro (robot description, xacro)
@@ -246,4 +246,32 @@
     </visual>
   </link>
+  <joint name="conveyor_joint" type="fixed">
+    <origin xyz="0 0 0" rpy="0 0 0" />
+    <parent link="base_link"/>
+    <child link="conveyor_link" />
+  </joint>
+  <link name="conveyor_link">
+  <collision>
+    <origin xyz="0 0 0.37" rpy="0 0 0"/>
+    <geometry>
+      <box size="1 0.7 0.1"/>
+    </geometry>
+  </collision>
+  <visual>
+    <origin xyz="0 0 0.37" rpy="0 0 0"/>
+    <geometry>
+      <box size="1 0.7 0.1"/>
+    </geometry>
+     <material name="white" />
+  </visual>
+  <inertial>
+    <origin xyz="0 0 0.1" rpy="0 0 0"/>
+    <mass value="1"/>
+    <inertia
+      ixx="1.0" ixy="0.0" ixz="0.0"
+      iyy="1.0" iyz="0.0"
+      izz="1.0"/>
+  </inertial>
+ </link>
   <link name="imu_link">
     <inertial>
